File: C05-22mini/kicad/PCB_DOWN/22miniD.sch (KiCad schematic (older format))
At the start: 78 parts, among them J1 DC_IN, J10 Sync-OUT, J11 4021/7219DOWN, J12 4021/7219UP, J13 AUX BUS UP, J14 AUX BUS DOWN, J2 D3, J3 TXRX, J4 ANALOGS, J5 SERVO1, J6 SERVO2, J7 OUT1, J8 OUT2, J9 Sync-IN, Q1 PN2222A, SW1 TR01, SW10 OFFBEAT, SW11 SYNCSEL, SW2 TR02, SW3 MUTE, SW4 ON/OFF, SW5 ST01, SW6 ST02, SW7 PLAY/PAUSE/CLEAR, SW8 ST03, SW9 ST04, U1 4021, U2 MAX7219, U3 L7805, U4 L7805

Commit message: actualizado pcb down
Connections:
- net GND: now also D22.2 (A), Q1.1 (E)
Changed lines of the file:
@@
 	13900 5200 13900 5050
 Wire Wire Line
-	13400 5200 13400 5150
+	13400 5150 13400 5300
 Wire Wire Line
 	13400 4600 13400 4850
@@
 Connection ~ 17000 5250
 NoConn ~ 2350 1350
+$Comp
+L GND #PWR?
+U 1 1 5BC74D8A
+P 13400 5300
+F 0 "#PWR?" H 13400 5050 50  0001 C CNN
+F 1 "GND" H 13400 5150 50  0000 C CNN
+F 2 "" H 13400 5300 50  0001 C CNN
+F 3 "" H 13400 5300 50  0001 C CNN
+	1    13400 5300
+	1    0    0    -1
+$EndComp
+Connection ~ 13400 5200
 $EndSCHEMATC
