File: C05-22mini/kicad/PCB_DOWN/22miniD.kicad_pcb (KiCad board)
At the start: 2 copper layers, 111 x 60 mm, 37 parts, among them J1 DC_IN, J10 Sync-OUT, J11 4021/7219DOWN, J14 AUX BUS DOWN, J2 D3, J3 TXRX, J4 ANALOGS, J5 SERVO1, J6 SERVO2, J7 OUT1, J8 OUT2, J9 Sync-IN, Q1 PN2222A, SW11 SYNCSEL, SW4 ON/OFF, U3 L7805, U4 L7805

Commit message: actualizado pcb down
Parts:
- C3: footprint Capacitors_THT:CP_Radial_D8.0mm_P3.80mm -> Capacitors_THT:CP_Radial_D5.0mm_P2.50mm
- C4: footprint Capacitors_THT:CP_Radial_D7.5mm_P2.50mm -> Capacitors_THT:CP_Radial_D5.0mm_P2.50mm
- C6: footprint Capacitors_THT:CP_Radial_D8.0mm_P3.80mm -> Capacitors_THT:CP_Radial_D8.0mm_P3.50mm
- moved G*** 0.84 mm to (86.9, 59.0)
- turned REF** to 0 degrees (x5)
Connections:
- D22 pad 2: Net-(D22-Pad2) -> GND
- Q1 pad 1: Net-(D22-Pad2) -> GND
Routing:
- net Net-(D22-Pad2): track 13.4 -> 0.00 mm, vias 1 -> 0
- net GND: track 277.5 -> 290.8 mm, vias 72 -> 73
Other:
- board text added: "pcb v2"

Commit message: crear images, gerbrs 22mini
Parts:
- added REF**: Pin_Header_Straight_1x04_Pitch2.54mm, Pin_Headers:Pin_Header_Straight_1x04_Pitch2.54mm, F.Cu at (131.7, 77.3)
- C3, C6: moved to B.Cu
- Q1: footprint TO_SOT_Packages_THT:TO-92_Inline_Narrow_Oval -> TO_SOT_Packages_THT:TO-92_Inline_Wide
- moved G*** 2.06 mm to (87.0, 61.0)
- moved Q1 0.54 mm to (92.1, 74.1)
Routing:
- net Net-(D22-Pad1): track 76.1 -> 83.3 mm
- net Net-(ARDUINO1-Pad21): track 64.4 -> 69.8 mm
- net +5V: track 61.6 -> 63.3 mm
- net Net-(ARDUINO1-Pad15): track 79.7 -> 80.7 mm
- net GND: track 290.8 -> 291.4 mm
Other:
- board text added: "GND"
