File: C05-22mini/kicad/PCB_UP/22mini.kicad_pcb (KiCad board)
At the start: 2 copper layers, 111 x 60 mm, 55 parts, among them J12 4021/7219UP, J13 AUX BUS UP, SW1 TR01, SW10 OFFBEAT, SW2 TR02, SW3 MUTE, SW5 ST01, SW6 ST02, SW7 PLAY/PAUSE/CLEAR, SW8 ST03, SW9 ST04, U1 4021, U2 MAX7219

Commit message: actualizado pcb down
Parts:
- moved REF** 0.75 mm to (33.2, 62.2)
Changed lines of the file:
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@@
   )
   (module Mounting_Holes:MountingHole_3.2mm_M3 (layer F.Cu)
-    (at 33.25 63)
+    (at 33.25 62.25)
     (descr "Mounting Hole 3.2mm, no annular, M3")
     (tags "mounting hole 3.2mm no annular m3")
